File: Kicad/Circuits-Imprimés/Module_0-Commutation_PTT-BITX40/Module_0-Commutation_PTT-BITX40.kicad_pcb (KiCad board)
At the start: 2 copper layers, 172.9 x 100.8 mm, 32 parts, among them J1 Conn_01x02, J10 Conn_01x02, J11 Conn_Coaxial, J12 Conn_Coaxial, J13 Conn_01x02, J14 Conn_01x02, J15 Conn_01x02, J16 Conn_01x03, J2 Conn_01x02, J3 Conn_Coaxial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

Commit message: Update project BITX 40
Update project BITX 40
Parts:
- removed REF** (x4): M3-Hole, Visserie-Trous-Modules:M3-Hole
- moved R4 177.7 mm to (320.2, 46.7)
- moved R3 171.5 mm to (309.9, 54.2)
- moved C1 157.7 mm to (328.1, 48.8)
- moved J13 148.4 mm to (303.9, 51.6)
- moved J5 147.1 mm to (271.5, 38.7)
- moved J6 139.5 mm to (271.5, 50.7)
- moved J14 132.4 mm to (317.1, 39.2)
- moved J9 130.0 mm to (311.0, 39.2)
- moved C2 129.8 mm to (305.5, 65.0)
- moved R2 128.6 mm to (328.1, 34.3)
- moved D1 121.5 mm to (288.1, 34.5)
- moved J8 118.4 mm to (255.2, 62.7)
- moved Q1 117.5 mm to (312.1, 50.3)
- moved J16 116.9 mm to (255.2, 50.7)
- moved J4 111.9 mm to (265.4, 39.2)
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Connections:
- K1 pad 11: Net-(K1-Pad11) -> (no net)
- K1 pad 13: Net-(J3-Pad1) -> (no net)
- K1 pad 4: (no net) -> Net-(J3-Pad1)
- K1 pad 6: (no net) -> Net-(K1-Pad6)
- K1 pad 8: (no net) -> Net-(J7-Pad1)
- K1 pad 9: Net-(J7-Pad1) -> (no net)
- K2 pad 11: Net-(K1-Pad11) -> Net-(K1-Pad6)
Routing:
- net TX: track 150.1 -> 0.00 mm
- net RX: track 95.1 -> 0.00 mm
- net 12V: track 76.5 -> 10.8 mm
- net Net-(K1-Pad6): track 0.00 -> 51.0 mm
- net Net-(K1-Pad11): track 31.3 -> 0.00 mm
- net Net-(C3-Pad1): track 27.0 -> 0.00 mm
- net Net-(J12-Pad1): track 24.2 -> 39.6 mm
- net Net-(J11-Pad1): track 10.5 -> 24.7 mm
- net Net-(Q1-Pad2): track 12.0 -> 0.00 mm
- net Net-(J7-Pad1): track 10.5 -> 19.7 mm
- net PTT: track 6.88 -> 0.00 mm
- net LedTX: track 6.35 -> 0.00 mm
- net LedRX: track 6.35 -> 0.00 mm
- net Net-(J3-Pad1): track 19.1 -> 19.7 mm
- removed copper zone on B.Cu, net GND
Other:
- board size 172.9 x 100.8 mm -> 75 x 65 mm
- net class Default: clearance 0.2 -> 0.3; trace_width 0.25 -> 1; via_dia 0.6 -> 1; via_drill 0.4 -> 0.8
- rule trace_clearance: 0.2 -> 0.3

Commit message: Update project BITX
Update project BITX 40. Add new hole. New version PCB.
Parts:
- added REF**: M3-Hole, Visserie-Trous-Modules:M3-Hole, F.Cu at (100.0, 60.0)
- added REF**: M3-Hole, Visserie-Trous-Modules:M3-Hole, F.Cu at (205.0, 60.0)
- added REF**: M3-Hole, Visserie-Trous-Modules:M3-Hole, F.Cu at (205.0, 120.0)
- added REF**: M3-Hole, Visserie-Trous-Modules:M3-Hole, F.Cu at (100.0, 120.0)
- J1, J10, J11, J12, J13, J14, J15, J2, J3, J7, J9: footprint Connectors:bornier2 -> Raccordement-Filaires:Connect-2pin
- J16, J4, J5, J6, J8: footprint Connectors:bornier3 -> Raccordement-Filaires:Connect-3pin
- moved C1 229.9 mm to (100.3, 80.0), turned to 0 degrees
- moved J14 224.8 mm to (97.8, 88.9)
- moved J9 222.9 mm to (97.8, 104.1), turned to 0 degrees
- moved J2 185.2 mm to (97.8, 111.8), turned to 0 degrees
- moved J15 183.0 mm to (97.8, 96.5)
- moved R2 170.3 mm to (167.6, 91.4)
- moved C2 164.6 mm to (142.2, 86.4), turned to 90 degrees
- moved D1 159.6 mm to (137.2, 86.4), turned to 90 degrees
- moved Q1 158.2 mm to (160.0, 94.0), turned to 0 degrees
- moved J1 151.9 mm to (161.3, 111.8)
- moved R4 150.7 mm to (180.3, 102.9), turned to 90 degrees
- moved C3 143.8 mm to (154.9, 86.4), turned to 90 degrees
- moved R3 142.0 mm to (176.5, 102.9), turned to 90 degrees
- moved R1 131.0 mm to (161.3, 99.1), turned to 270 degrees
- moved J13 119.5 mm to (200.7, 111.8), turned to 0 degrees
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Routing:
- net TX: track 0.00 -> 134.0 mm
- net 12V: track 10.8 -> 137.9 mm
- net RX: track 0.00 -> 69.3 mm
- net Net-(C3-Pad1): track 0.00 -> 23.9 mm
- net Net-(J12-Pad1): track 39.6 -> 16.5 mm
- net GND: track 0.00 -> 22.9 mm
- net Net-(K1-Pad6): track 51.0 -> 73.7 mm
- net Net-(Q1-Pad2): track 0.00 -> 10.2 mm
- net LedRX: track 0.00 -> 9.42 mm
- net LedTX: track 0.00 -> 8.89 mm
- net Net-(J11-Pad1): track 24.7 -> 16.5 mm
- net PTT: track 0.00 -> 5.08 mm
- added copper zone on B.Cu, net GND
Other:
- board size 75 x 65 mm -> 121.9 x 76.2 mm
- net class Default: clearance 0.3 -> 0.2
- net class TX/RX: clearance 0.3 -> 0.2
- rule trace_clearance: 0.3 -> 0.2
- board text added: "Ant"
- board text added: "BITX 40 Module 0"
- board text added: "F4HYU F1HSU"
- board text added: "Mod 1"
- board text added: "Mod 10"
- board text added: "Mod 12"
