File: Kicad/Circuits-Imprimés/Module_0-Commutation_PTT-BITX40/Module_0-Commutation_PTT-BITX40.kicad_pcb (KiCad board)
At the start: 2 copper layers, 121.9 x 76.2 mm, 32 parts, among them J1 Conn_01x02, J10 Conn_01x02, J11 Conn_Coaxial, J12 Conn_Coaxial, J13 Conn_01x02, J14 Conn_01x02, J15 Conn_01x02, J16 Conn_01x03, J2 Conn_01x02, J3 Conn_Coaxial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

Commit message: Update
Update
Other:
- net class Default: clearance 0.2 -> 0.3
- net class TX/RX: clearance 0.2 -> 0.3
- rule trace_clearance: 0.2 -> 0.3
Changed lines of the file:
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@@
     (user_trace_width 1.5)
     (user_trace_width 2)
-    (trace_clearance 0.2)
+    (trace_clearance 0.3)
     (zone_clearance 0.508)
     (zone_45_only no)
@@
   (net 14 "Net-(K1-Pad6)")
   (net_class Default "Ceci est la Netclass par défaut"
-    (clearance 0.2)
+    (clearance 0.3)
     (trace_width 1)
     (via_dia 1)
@@
   )
   (net_class TX/RX ""
-    (clearance 0.2)
+    (clearance 0.3)
     (trace_width 0.5)
     (via_dia 1)
@@
   (gr_line (start 91.44 127) (end 213.36 127) (angle 90) (layer Edge.Cuts) (width 0.15))
   (gr_line (start 91.44 50.8) (end 91.44 127) (angle 90) (layer Edge.Cuts) (width 0.15))
-  (gr_text "F4HYU\nF1HSU" (at 143.51 104.14) (layer B.Cu)
+  (gr_text "F4HYU\nF1HSU" (at 143.51 104.14) (layer F.SilkS)
     (effects (font (size 3 3) (thickness 0.6)) (justify mirror))
   )
-  (gr_text "BITX 40\nModule 0" (at 121.92 104.14) (layer B.Cu)
+  (gr_text "BITX 40\nModule 0" (at 121.92 104.14) (layer F.SilkS)
     (effects (font (size 3 3) (thickness 0.6)) (justify mirror))
   )
