File: Kicad/Circuits-Imprimés/Module_0-Commutation_PTT-BITX40/Module_0-Commutation_PTT-BITX40.sch (KiCad schematic (older format))
At the start: 28 parts, among them J1 Conn_01x02, J10 Conn_01x02, J11 Conn_Coaxial, J12 Conn_Coaxial, J13 Conn_01x02, J14 Conn_01x02, J15 Conn_01x02, J16 Conn_01x03, J2 Conn_01x02, J3 Conn_Coaxial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

Commit message: Update project BITX 40
Update project BITX 40
Connections:
- net at K1.11: no longer K2.11
- net at K1.13: no longer J3.1 (In)
- net at K1.4: now also J3.1 (In)
- net at K1.6: now also K2.11
- net at K1.8: now also J7.1 (In)
- net at K1.9: no longer J7.1 (In)
Other:
- moved on the sheet: J3
Changed lines of the file:
@@
 L Conn_Coaxial J3
 U 1 1 5A7E0CD8
-P 1600 2000
-F 0 "J3" H 1610 2120 50  0000 C CNN
-F 1 "Conn_Coaxial" V 1715 2000 50  0000 C CNN
-F 2 "Connectors:bornier2" H 1600 2000 50  0001 C CNN
-F 3 "" H 1600 2000 50  0001 C CNN
-	1    1600 2000
+P 1850 2400
+F 0 "J3" H 1860 2520 50  0000 C CNN
+F 1 "Conn_Coaxial" V 1965 2400 50  0000 C CNN
+F 2 "Connectors:bornier2" H 1850 2400 50  0001 C CNN
+F 3 "" H 1850 2400 50  0001 C CNN
+	1    1850 2400
 	-1   0    0    -1
 $EndComp
-Text Notes 1250 1650 0    60   ~ 0
+Text Notes 1500 2050 0    60   ~ 0
 Vers l'antenne
 $Comp
@@
 L GND #PWR04
 U 1 1 5A7E10DE
-P 1600 2350
-F 0 "#PWR04" H 1600 2100 50  0001 C CNN
-F 1 "GND" H 1600 2200 50  0000 C CNN
-F 2 "" H 1600 2350 50  0001 C CNN
-F 3 "" H 1600 2350 50  0001 C CNN
-	1    1600 2350
+P 1850 2750
+F 0 "#PWR04" H 1850 2500 50  0001 C CNN
+F 1 "GND" H 1850 2600 50  0000 C CNN
+F 2 "" H 1850 2750 50  0001 C CNN
+F 3 "" H 1850 2750 50  0001 C CNN
+	1    1850 2750
 	1    0    0    -1
 $EndComp
@@
 LedTX
 Wire Wire Line
-	1750 2000 2650 2000
-Wire Wire Line
-	3250 1900 3400 1900
-Wire Wire Line
-	3400 1900 3400 1100
-Wire Wire Line
 	3400 1100 3600 1100
 Wire Wire Line
@@
 	3750 1300 3750 1450
 Wire Wire Line
-	1600 2200 1600 2350
-Wire Notes Line
-	1200 1500 1950 1500
-Wire Notes Line
-	1950 1500 1950 2600
-Wire Notes Line
-	1950 2600 1200 2600
-Wire Notes Line
-	1200 2600 1200 1500
+	1850 2600 1850 2750
+Wire Notes Line
+	1450 1900 2200 1900
+Wire Notes Line
+	2200 1900 2200 3000
+Wire Notes Line
+	2200 3000 1450 3000
+Wire Notes Line
+	1450 3000 1450 1900
 Wire Notes Line
 	3350 550  3350 1650
@@
 Connection ~ 7350 4050
 Wire Wire Line
-	3250 2100 6600 2100
-Wire Wire Line
 	6000 1100 6000 1900
 Wire Wire Line
@@
 Wire Wire Line
 	8450 2400 8900 2400
+Wire Wire Line
+	2000 2400 2650 2400
+Wire Wire Line
+	3400 1100 3400 2300
+Wire Wire Line
+	3400 2300 3250 2300
+Wire Wire Line
+	3250 2500 5350 2500
+Wire Wire Line
+	5350 2500 5350 2100
+Wire Wire Line
+	5350 2100 6600 2100
 $EndSCHEMATC

Commit message: Update project BITX
Update project BITX 40. Add new hole. New version PCB.
Parts:
- J1, J10, J11, J12, J13, J14, J15, J2, J3, J7, J9: footprint Connectors:bornier2 -> Raccordement-Filaires:Connect-2pin
- J16, J4, J5, J6, J8: footprint Connectors:bornier3 -> Raccordement-Filaires:Connect-3pin
Changed lines of the file:
@@
 F 0 "J3" H 1860 2520 50  0000 C CNN
 F 1 "Conn_Coaxial" V 1965 2400 50  0000 C CNN
-F 2 "Connectors:bornier2" H 1850 2400 50  0001 C CNN
+F 2 "Raccordement-Filaires:Connect-2pin" H 1850 2400 50  0001 C CNN
 F 3 "" H 1850 2400 50  0001 C CNN
 	1    1850 2400
@@
 F 0 "J7" H 3760 1220 50  0000 C CNN
 F 1 "Conn_Coaxial" V 3865 1100 50  0000 C CNN
-F 2 "Connectors:bornier2" H 3750 1100 50  0001 C CNN
+F 2 "Raccordement-Filaires:Connect-2pin" H 3750 1100 50  0001 C CNN
 F 3 "" H 3750 1100 50  0001 C CNN
 	1    3750 1100
@@
 F 0 "J11" H 5760 1220 50  0000 C CNN
 F 1 "Conn_Coaxial" V 5865 1100 50  0000 C CNN
-F 2 "Connectors:bornier2" H 5750 1100 50  0001 C CNN
+F 2 "Raccordement-Filaires:Connect-2pin" H 5750 1100 50  0001 C CNN
 F 3 "" H 5750 1100 50  0001 C CNN
 	1    5750 1100
@@
 F 0 "J12" H 9060 2520 50  0000 C CNN
 F 1 "Conn_Coaxial" V 9165 2400 50  0000 C CNN
-F 2 "Connectors:bornier2" H 9050 2400 50  0001 C CNN
+F 2 "Raccordement-Filaires:Connect-2pin" H 9050 2400 50  0001 C CNN
 F 3 "" H 9050 2400 50  0001 C CNN
 	1    9050 2400
@@
 F 0 "J2" H 1000 6350 50  0000 C CNN
 F 1 "Conn_01x02" H 1000 6050 50  0000 C CNN
-F 2 "Connectors:bornier2" H 1000 6250 50  0001 C CNN
+F 2 "Raccordement-Filaires:Connect-2pin" H 1000 6250 50  0001 C CNN
 F 3 "" H 1000 6250 50  0001 C CNN
 	1    1000 6250
@@
 F 0 "J1" H 1000 5450 50  0000 C CNN
 F 1 "Conn_01x02" H 1000 5150 50  0000 C CNN
-F 2 "Connectors:bornier2" H 1000 5350 50  0001 C CNN
+F 2 "Raccordement-Filaires:Connect-2pin" H 1000 5350 50  0001 C CNN
 F 3 "" H 1000 5350 50  0001 C CNN
 	1    1000 5350
@@
 F 0 "J4" H 3350 5600 50  0000 C CNN
 F 1 "Conn_01x03" H 3350 5200 50  0000 C CNN
-F 2 "Connectors:bornier3" H 3350 5400 50  0001 C CNN
+F 2 "Raccordement-Filaires:Connect-3pin" H 3350 5400 50  0001 C CNN
 F 3 "" H 3350 5400 50  0001 C CNN
 	1    3350 5400
@@
 F 0 "J5" H 3350 6450 50  0000 C CNN
 F 1 "Conn_01x03" H 3350 6050 50  0000 C CNN
-F 2 "Connectors:bornier3" H 3350 6250 50  0001 C CNN
+F 2 "Raccordement-Filaires:Connect-3pin" H 3350 6250 50  0001 C CNN
 F 3 "" H 3350 6250 50  0001 C CNN
 	1    3350 6250
@@
 F 0 "J6" H 3350 7300 50  0000 C CNN
 F 1 "Conn_01x03" H 3350 6900 50  0000 C CNN
-F 2 "Connectors:bornier3" H 3350 7100 50  0001 C CNN
+F 2 "Raccordement-Filaires:Connect-3pin" H 3350 7100 50  0001 C CNN
 F 3 "" H 3350 7100 50  0001 C CNN
 	1    3350 7100
@@
 F 0 "J14" H 9150 5300 50  0000 C CNN
 F 1 "Conn_01x02" H 9150 5000 50  0000 C CNN
-F 2 "Connectors:bornier2" H 9150 5200 50  0001 C CNN
+F 2 "Raccordement-Filaires:Connect-2pin" H 9150 5200 50  0001 C CNN
 F 3 "" H 9150 5200 50  0001 C CNN
 	1    9150 5200
@@
 F 0 "J15" H 9150 6050 50  0000 C CNN
 F 1 "Conn_01x02" H 9150 5750 50  0000 C CNN
-F 2 "Connectors:bornier2" H 9150 5950 50  0001 C CNN
+F 2 "Raccordement-Filaires:Connect-2pin" H 9150 5950 50  0001 C CNN
 F 3 "" H 9150 5950 50  0001 C CNN
 	1    9150 5950
@@
 F 0 "J13" H 9150 4600 50  0000 C CNN
 F 1 "Conn_01x02" H 9150 4300 50  0000 C CNN
-F 2 "Connectors:bornier2" H 9150 4500 50  0001 C CNN
+F 2 "Raccordement-Filaires:Connect-2pin" H 9150 4500 50  0001 C CNN
 F 3 "" H 9150 4500 50  0001 C CNN
 	1    9150 4500
@@
 F 0 "J8" H 5400 7300 50  0000 C CNN
 F 1 "Conn_01x03" H 5400 6900 50  0000 C CNN
-F 2 "Connectors:bornier3" H 5400 7100 50  0001 C CNN
+F 2 "Raccordement-Filaires:Connect-3pin" H 5400 7100 50  0001 C CNN
 F 3 "" H 5400 7100 50  0001 C CNN
 	1    5400 7100
@@
 F 0 "J10" H 5450 6100 50  0000 C CNN
 F 1 "Conn_01x02" H 5450 5800 50  0000 C CNN
-F 2 "Connectors:bornier2" H 5450 6000 50  0001 C CNN
+F 2 "Raccordement-Filaires:Connect-2pin" H 5450 6000 50  0001 C CNN
 F 3 "" H 5450 6000 50  0001 C CNN
 	1    5450 6000
@@
 F 0 "J9" H 5450 5400 50  0000 C CNN
 F 1 "Conn_01x02" H 5450 5100 50  0000 C CNN
-F 2 "Connectors:bornier2" H 5450 5300 50  0001 C CNN
+F 2 "Raccordement-Filaires:Connect-2pin" H 5450 5300 50  0001 C CNN
 F 3 "" H 5450 5300 50  0001 C CNN
 	1    5450 5300
@@
 F 0 "J16" H 9250 4000 50  0000 C CNN
 F 1 "Conn_01x03" H 9250 3600 50  0000 C CNN
-F 2 "Connectors:bornier3" H 9250 3800 50  0001 C CNN
+F 2 "Raccordement-Filaires:Connect-3pin" H 9250 3800 50  0001 C CNN
 F 3 "" H 9250 3800 50  0001 C CNN
 	1    9250 3800
