File: Kicad/Circuits-Imprimés/Module_1-Filtre_TX-RX-BITX40/Module_1-Filtre_TX-RX-BITX40.kicad_pcb (KiCad board)
At the start: 2 copper layers, 104.1 x 33 mm, 16 parts, among them J1 Conn_Coaxial, J2 Conn_Coaxial

Commit message: Update
Update
Changed lines of the file:
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@@
     (pad 1 thru_hole circle (at 0 0) (size 3 3) (drill 1) (layers *.Cu *.Mask))
   )
-  (gr_text "F4HYU F1HSU" (at 109.22 53.34) (layer B.Cu)
+  (gr_text "F4HYU F1HSU" (at 109.22 53.34) (layer F.SilkS)
     (effects (font (size 3 3) (thickness 0.3)) (justify mirror))
   )
-  (gr_text "Module 1 Filtre TX / RX" (at 109.22 76.2) (layer B.Cu)
+  (gr_text "Module 1 Filtre TX / RX" (at 109.22 76.2) (layer F.SilkS)
     (effects (font (size 3 3) (thickness 0.3)) (justify mirror))
   )
