File: Kicad/Circuits-Imprimés/Module_2-1_2_3-Amplificateur-Bi-Directionnel-BITX40/Module_2-1_2_3-Amplificateur-Bi-Directionnel-BITX40.kicad_pcb (KiCad board)
At the start: 2 copper layers, 50 x 85 mm, 31 parts, among them J1 Conn_01x03, J2 Conn_01x02, J3 Conn_01x02, Q1 2N3904, Q2 2N3904

Commit message: Update
Update
Parts:
- moved C1 77.1 mm to (170.2, 76.2)
- moved Q1 75.9 mm to (175.3, 77.5)
- moved C7 75.5 mm to (182.9, 76.2)
- moved R5 75.5 mm to (175.3, 71.1)
- moved R2 74.0 mm to (162.6, 86.4), turned to 90 degrees
- moved C3 71.9 mm to (170.2, 81.3)
- moved R8 65.5 mm to (175.3, 86.4), turned to 90 degrees
- moved D1 59.0 mm to (63.5, 89.4)
- moved R4 54.2 mm to (96.6, 89.2)
- moved J3 50.4 mm to (67.0, 102.2), turned to 180 degrees
- moved REF** 49.7 mm to (106.7, 111.7)
- moved REF** 46.2 mm to (107.5, 104.4)
- moved C5 46.2 mm to (105.5, 97.2)
- moved R6 43.3 mm to (85.8, 101.2)
- moved REF** 43.3 mm to (112.2, 97.1)
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Routing:
- net RX: track 68.9 -> 0.00 mm
- net TX: track 38.4 -> 0.00 mm
- net Net-(C1-Pad2): track 30.5 -> 0.00 mm
- net Net-(C7-Pad1): track 30.5 -> 0.00 mm
- net Net-(C2-Pad1): track 16.5 -> 0.00 mm
- net Net-(C1-Pad1): track 15.8 -> 0.00 mm
- net Net-(C8-Pad2): track 15.3 -> 0.00 mm
- net Net-(C7-Pad2): track 15.3 -> 0.00 mm
- net Net-(C6-Pad2): track 14.0 -> 0.00 mm
- net Net-(C3-Pad1): track 11.4 -> 0.00 mm
- net Net-(C5-Pad2): track 8.93 -> 0.00 mm
- net Net-(C4-Pad2): track 8.93 -> 0.00 mm
- net Net-(D2-Pad2): track 6.13 -> 0.00 mm
- net Net-(D1-Pad2): track 6.13 -> 0.00 mm
- net Net-(C3-Pad2): track 3.85 -> 0.00 mm
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- removed copper zone on B.Cu, net GND
- removed copper zone on F.Cu, net GND
Other:
- board outline removed
