File: Kicad/Module_0-Commutation_PTT-BITX40/Module_0-Commutation_PTT-BITX40.sch (KiCad schematic (older format))
At the start: 41 parts, among them J1 Conn_01x02, J10 Conn_Coaxial, J11 Conn_Coaxial, J12 Conn_01x02, J13 Conn_01x02, J14 Conn_01x02, J15 Conn_01x02, J16 Conn_01x02, J17 Conn_Coaxial, J18 Conn_01x03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

Commit message: Update missing PTT-
Missing PNP mount PTT- are changed
PTT+ not use GND. Update for the 12V command.
Connections:
- net 12V: now also J1.1 (Pin_1)
- net GND: now also Q2.2 (C); no longer J1.2 (Pin_2), Q2.3 (E)
- net at R1.2: now also J1.2 (Pin_2); no longer J1.1 (Pin_1)
- net at SW3.1: now also Q2.3 (E); no longer Q2.2 (C)
Other:
- moved on the sheet: J1, SW3
Changed lines of the file:
@@
 L Conn_01x02 J1
 U 1 1 5AB51015
-P 950 5350
-F 0 "J1" H 950 5450 50  0000 C CNN
-F 1 "Conn_01x02" H 950 5150 50  0000 C CNN
-F 2 "alex-library:Connect-2pin" H 950 5350 50  0001 C CNN
-F 3 "" H 950 5350 50  0001 C CNN
-	1    950  5350
+P 950 5250
+F 0 "J1" H 950 5350 50  0000 C CNN
+F 1 "Conn_01x02" H 950 5050 50  0000 C CNN
+F 2 "alex-library:Connect-2pin" H 950 5250 50  0001 C CNN
+F 3 "" H 950 5250 50  0001 C CNN
+	1    950  5250
 	-1   0    0    -1
 $EndComp
 Text Notes 650  5400 0    60   ~ 0
 PTT+
-Text Notes 650  5500 0    60   ~ 0
-GND
+Text Notes 650  5300 0    60   ~ 0
++12V
 $Comp
 L Conn_01x02 J3
@@
 $Comp
 L GND #PWR05
-U 1 1 5AB518C9
-P 1300 5500
-F 0 "#PWR05" H 1300 5250 50  0001 C CNN
-F 1 "GND" H 1300 5350 50  0000 C CNN
-F 2 "" H 1300 5500 50  0001 C CNN
-F 3 "" H 1300 5500 50  0001 C CNN
-	1    1300 5500
-	1    0    0    -1
-$EndComp
-$Comp
-L GND #PWR06
 U 1 1 5AB51A08
 P 1450 1250
-F 0 "#PWR06" H 1450 1000 50  0001 C CNN
+F 0 "#PWR05" H 1450 1000 50  0001 C CNN
 F 1 "GND" H 1450 1100 50  0000 C CNN
 F 2 "" H 1450 1250 50  0001 C CNN
@@
 $EndComp
 $Comp
-L GND #PWR07
+L GND #PWR06
 U 1 1 5AB51A3D
 P 1900 1600
-F 0 "#PWR07" H 1900 1350 50  0001 C CNN
+F 0 "#PWR06" H 1900 1350 50  0001 C CNN
 F 1 "GND" H 1900 1450 50  0000 C CNN
 F 2 "" H 1900 1600 50  0001 C CNN
@@
 $EndComp
 $Comp
-L GND #PWR08
+L GND #PWR07
 U 1 1 5AB51A72
 P 2250 1600
-F 0 "#PWR08" H 2250 1350 50  0001 C CNN
+F 0 "#PWR07" H 2250 1350 50  0001 C CNN
 F 1 "GND" H 2250 1450 50  0000 C CNN
 F 2 "" H 2250 1600 50  0001 C CNN
@@
 PTT
 $Comp
-L GND #PWR09
+L GND #PWR08
 U 1 1 5AB53127
 P 3050 4150
-F 0 "#PWR09" H 3050 3900 50  0001 C CNN
+F 0 "#PWR08" H 3050 3900 50  0001 C CNN
 F 1 "GND" H 3050 4000 50  0000 C CNN
 F 2 "" H 3050 4150 50  0001 C CNN
@@
 $EndComp
 $Comp
-L GND #PWR010
+L GND #PWR09
 U 1 1 5AB5388B
 P 1750 5800
-F 0 "#PWR010" H 1750 5550 50  0001 C CNN
+F 0 "#PWR09" H 1750 5550 50  0001 C CNN
 F 1 "GND" H 1750 5650 50  0000 C CNN
 F 2 "" H 1750 5800 50  0001 C CNN
@@
 $EndComp
 $Comp
-L GND #PWR011
+L GND #PWR010
 U 1 1 5AB54507
 P 2200 5800
-F 0 "#PWR011" H 2200 5550 50  0001 C CNN
+F 0 "#PWR010" H 2200 5550 50  0001 C CNN
 F 1 "GND" H 2200 5650 50  0000 C CNN
 F 2 "" H 2200 5800 50  0001 C CNN
@@
 GND
 $Comp
-L GND #PWR012
+L GND #PWR011
 U 1 1 5AB55A5C
 P 1300 7050
-F 0 "#PWR012" H 1300 6800 50  0001 C CNN
+F 0 "#PWR011" H 1300 6800 50  0001 C CNN
 F 1 "GND" H 1300 6900 50  0000 C CNN
 F 2 "" H 1300 7050 50  0001 C CNN
@@
 $EndComp
 $Comp
-L GND #PWR013
+L GND #PWR012
 U 1 1 5AB55A6B
 P 1750 7350
-F 0 "#PWR013" H 1750 7100 50  0001 C CNN
+F 0 "#PWR012" H 1750 7100 50  0001 C CNN
 F 1 "GND" H 1750 7200 50  0000 C CNN
 F 2 "" H 1750 7350 50  0001 C CNN
@@
 $EndComp
 $Comp
-L GND #PWR014
+L GND #PWR013
 U 1 1 5AB55A7D
-P 2200 7350
-F 0 "#PWR014" H 2200 7100 50  0001 C CNN
-F 1 "GND" H 2200 7200 50  0000 C CNN
-F 2 "" H 2200 7350 50  0001 C CNN
-F 3 "" H 2200 7350 50  0001 C CNN
-	1    2200 7350
+P 2700 6600
+F 0 "#PWR013" H 2700 6350 50  0001 C CNN
+F 1 "GND" H 2700 6450 50  0000 C CNN
+F 2 "" H 2700 6600 50  0001 C CNN
+F 3 "" H 2700 6600 50  0001 C CNN
+	1    2700 6600
 	1    0    0    -1
 $EndComp
@@
 L Chevron SW3
 U 1 1 5AB55A83
-P 2550 6600
-F 0 "SW3" H 2550 6500 60  0000 C CNN
-F 1 "Chevron" H 2550 6700 60  0000 C CNN
-F 2 "alex-library:Chevron" H 2650 6600 60  0001 C CNN
-F 3 "" H 2650 6600 60  0001 C CNN
-	1    2550 6600
-	1    0    0    -1
-$EndComp
-Text GLabel 2950 6600 2    60   Input ~ 0
+P 2550 7200
+F 0 "SW3" H 2550 7100 60  0000 C CNN
+F 1 "Chevron" H 2550 7300 60  0000 C CNN
+F 2 "alex-library:Chevron" H 2650 7200 60  0001 C CNN
+F 3 "" H 2650 7200 60  0001 C CNN
+	1    2550 7200
+	1    0    0    -1
+$EndComp
+Text GLabel 2950 7200 2    60   Input ~ 0
 PTT
 $Comp
@@
 PTT
 $Comp
-L GND #PWR015
+L GND #PWR014
 U 1 1 5AB567F0
 P 1550 4300
-F 0 "#PWR015" H 1550 4050 50  0001 C CNN
+F 0 "#PWR014" H 1550 4050 50  0001 C CNN
 F 1 "GND" H 1550 4150 50  0000 C CNN
 F 2 "" H 1550 4300 50  0001 C CNN
@@
 TX\nRX\nGND\nVers Module 2-1
 $Comp
-L GND #PWR016
+L GND #PWR015
 U 1 1 5AB58B86
 P 3750 5100
-F 0 "#PWR016" H 3750 4850 50  0001 C CNN
+F 0 "#PWR015" H 3750 4850 50  0001 C CNN
 F 1 "GND" H 3750 4950 50  0000 C CNN
 F 2 "" H 3750 5100 50  0001 C CNN
@@
 TX\nRX\nGND\nVers Module 2-2
 $Comp
-L GND #PWR017
+L GND #PWR016
 U 1 1 5AB5995F
 P 3750 5850
-F 0 "#PWR017" H 3750 5600 50  0001 C CNN
+F 0 "#PWR016" H 3750 5600 50  0001 C CNN
 F 1 "GND" H 3750 5700 50  0000 C CNN
 F 2 "" H 3750 5850 50  0001 C CNN
@@
 TX\nRX\nGND\nVers Module 2-3
 $Comp
-L GND #PWR018
+L GND #PWR017
 U 1 1 5AB59B49
 P 3750 6600
-F 0 "#PWR018" H 3750 6350 50  0001 C CNN
+F 0 "#PWR017" H 3750 6350 50  0001 C CNN
 F 1 "GND" H 3750 6450 50  0000 C CNN
 F 2 "" H 3750 6600 50  0001 C CNN
@@
 TX\nRX\nGND\nVers Module 9
 $Comp
-L GND #PWR019
+L GND #PWR018
 U 1 1 5AB5A43E
 P 3750 7350
-F 0 "#PWR019" H 3750 7100 50  0001 C CNN
+F 0 "#PWR018" H 3750 7100 50  0001 C CNN
 F 1 "GND" H 3750 7200 50  0000 C CNN
 F 2 "" H 3750 7350 50  0001 C CNN
@@
 $EndComp
 $Comp
-L GND #PWR020
+L GND #PWR019
 U 1 1 5AB5A910
 P 10000 6200
-F 0 "#PWR020" H 10000 5950 50  0001 C CNN
+F 0 "#PWR019" H 10000 5950 50  0001 C CNN
 F 1 "GND" H 10000 6050 50  0000 C CNN
 F 2 "" H 10000 6200 50  0001 C CNN
@@
 $EndComp
 $Comp
-L GND #PWR021
+L GND #PWR020
 U 1 1 5AB5D291
 P 5900 5000
-F 0 "#PWR021" H 5900 4750 50  0001 C CNN
+F 0 "#PWR020" H 5900 4750 50  0001 C CNN
 F 1 "GND" H 5900 4850 50  0000 C CNN
 F 2 "" H 5900 5000 50  0001 C CNN
@@
 $EndComp
 $Comp
-L GND #PWR022
+L GND #PWR021
 U 1 1 5AB5E6C5
 P 5900 5550
-F 0 "#PWR022" H 5900 5300 50  0001 C CNN
+F 0 "#PWR021" H 5900 5300 50  0001 C CNN
 F 1 "GND" H 5900 5400 50  0000 C CNN
 F 2 "" H 5900 5550 50  0001 C CNN
@@
 $EndComp
 $Comp
-L GND #PWR023
+L GND #PWR022
 U 1 1 5AB5E772
 P 5900 6100
-F 0 "#PWR023" H 5900 5850 50  0001 C CNN
+F 0 "#PWR022" H 5900 5850 50  0001 C CNN
 F 1 "GND" H 5900 5950 50  0000 C CNN
 F 2 "" H 5900 6100 50  0001 C CNN
@@
 $EndComp
 $Comp
-L GND #PWR024
+L GND #PWR023
 U 1 1 5AB5E829
 P 7850 5000
-F 0 "#PWR024" H 7850 4750 50  0001 C CNN
+F 0 "#PWR023" H 7850 4750 50  0001 C CNN
 F 1 "GND" H 7850 4850 50  0000 C CNN
 F 2 "" H 7850 5000 50  0001 C CNN
@@
 $EndComp
 $Comp
-L GND #PWR025
+L GND #PWR024
 U 1 1 5AB5EA6D
 P 7850 5550
-F 0 "#PWR025" H 7850 5300 50  0001 C CNN
+F 0 "#PWR024" H 7850 5300 50  0001 C CNN
 F 1 "GND" H 7850 5400 50  0000 C CNN
 F 2 "" H 7850 5550 50  0001 C CNN
@@
 $EndComp
 $Comp
-L GND #PWR026
+L GND #PWR025
 U 1 1 5AB63761
 P 9450 5150
-F 0 "#PWR026" H 9450 4900 50  0001 C CNN
+F 0 "#PWR025" H 9450 4900 50  0001 C CNN
 F 1 "GND" H 9450 5000 50  0000 C CNN
 F 2 "" H 9450 5150 50  0001 C CNN
@@
 $EndComp
 $Comp
-L GND #PWR027
+L GND #PWR026
 U 1 1 5AB63825
 P 9700 5150
-F 0 "#PWR027" H 9700 4900 50  0001 C CNN
+F 0 "#PWR026" H 9700 4900 50  0001 C CNN
 F 1 "GND" H 9700 5000 50  0000 C CNN
 F 2 "" H 9700 5150 50  0001 C CNN
@@
 $EndComp
 $Comp
-L GND #PWR028
+L GND #PWR027
 U 1 1 5AB6389F
 P 9950 5150
-F 0 "#PWR028" H 9950 4900 50  0001 C CNN
+F 0 "#PWR027" H 9950 4900 50  0001 C CNN
 F 1 "GND" H 9950 5000 50  0000 C CNN
 F 2 "" H 9950 5150 50  0001 C CNN
@@
 $EndComp
 $Comp
-L GND #PWR029
+L GND #PWR028
 U 1 1 5AB63919
 P 10200 5150
-F 0 "#PWR029" H 10200 4900 50  0001 C CNN
+F 0 "#PWR028" H 10200 4900 50  0001 C CNN
 F 1 "GND" H 10200 5000 50  0000 C CNN
 F 2 "" H 10200 5150 50  0001 C CNN
@@
 Connection ~ 2250 1100
 Wire Wire Line
-	1150 5450 1300 5450
-Wire Wire Line
-	1300 5450 1300 5500
-Wire Wire Line
 	7600 2400 10000 2400
 Wire Wire Line
@@
 	1750 5350 1750 5400
 Connection ~ 1750 5350
-Wire Wire Line
-	1350 5350 1150 5350
 Wire Notes Line
 	550  4700 3250 4700
@@
 	1300 7000 1300 7050
 Wire Wire Line
-	2950 6600 2850 6600
+	2950 7200 2850 7200
 Wire Wire Line
 	1750 7250 1750 7350
@@
 Wire Notes Line
 	550  7700 550  6250
-Wire Wire Line
-	2250 6600 2200 6600
-Wire Wire Line
-	2200 6600 2200 6700
 Wire Wire Line
 	1900 6900 1650 6900
@@
 	1750 6950 1750 6900
 Connection ~ 1750 6900
-Wire Wire Line
-	2200 7350 2200 7100
 Wire Wire Line
 	1400 4200 1550 4200
@@
 Wire Notes Line
 	9300 5400 9300 4700
+Wire Wire Line
+	2200 6700 2200 6500
+Wire Wire Line
+	2200 6500 2700 6500
+Wire Wire Line
+	2700 6500 2700 6600
+Wire Wire Line
+	2200 7100 2200 7200
+Wire Wire Line
+	2200 7200 2250 7200
+Text GLabel 1350 5150 2    60   Input ~ 0
+12V
+Wire Wire Line
+	1150 5250 1250 5250
+Wire Wire Line
+	1250 5250 1250 5150
+Wire Wire Line
+	1250 5150 1350 5150
+Wire Wire Line
+	1150 5350 1350 5350
 $EndSCHEMATC

Commit message: Commit
Commit
Parts:
- C1, C2, C4, C5, C6: symbol C -> Device:C
- C3: symbol CP -> Device:CP
- D1, D2: symbol D -> Device:D
- H1, H2, H3, H4: symbol M3-Hole -> alex-library:M3-Hole
- J1, J12, J13, J14, J15, J16, J2, J3, J4: symbol Conn_01x02 -> conn:Conn_01x02
- J10, J11, J17, J5: symbol Conn_Coaxial -> conn:Conn_Coaxial
- J18, J6, J7, J8, J9: symbol Conn_01x03 -> conn:Conn_01x03
- K1, K2: symbol D2n -> alex-library:D2n
- Q1: symbol Q_NPN_BCE -> Device:Q_NPN_BCE
- Q2: symbol Q_PNP_BCE -> Device:Q_PNP_BCE
- R1, R2, R3, R4: symbol R -> Device:R
- SW1, SW2, SW3: symbol Chevron -> Module_0-Commutation_PTT-BITX40-rescue:Chevron
