File: Kicad/Module_2-Amplificateur_bi_directionel_-BITX40-Mod_21_22_23/Module_2-Amplificateur_bi_directionel_-BITX40-Mod_21_22_23.kicad_pcb (KiCad board)
At the start: 2 copper layers, 60 x 50 mm, 31 parts, among them J1 Conn_01x03, J2 Conn_01x02, J3 Conn_01x02, Q1 2N2222a, Q2 2N2222a

Commit message: Update
Update
Parts:
- added G***: LOGO, logos:F4HYU-6x3-Logo, F.Cu at (175.0, 65.0)
- H1, H2, H3, H4: footprint alex-library:M3-Hole -> alex-library:M3-Real-Hole
- moved R2 40.7 mm to (118.1, 95.2), turned to 90 degrees
- moved Q1 19.1 mm to (148.6, 74.9)
- moved C4 16.2 mm to (123.2, 76.2), turned to 90 degrees
- moved H2 15.0 mm to (175.0, 95.0)
- moved H4 15.0 mm to (175.0, 55.0)
- moved D2 14.5 mm to (128.3, 82.5), turned to 270 degrees
- moved J2 13.0 mm to (111.8, 68.6), turned to 270 degrees
- moved J3 12.8 mm to (174.0, 82.5)
- moved R1 12.7 mm to (166.4, 55.9)
- moved R5 11.4 mm to (161.3, 71.1)
- moved R7 10.8 mm to (123.2, 80.0)
- moved C5 10.2 mm to (156.2, 91.4)
- moved C7 10.2 mm to (156.2, 78.7)
- moved C8 10.2 mm to (156.2, 82.5)
- moved D1 10.2 mm to (156.2, 68.6)
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Routing:
- net TX: track 18.3 -> 72.2 mm
- net Net-(C2-Pad1): track 35.7 -> 20.6 mm
- net Net-(C1-Pad1): track 15.0 -> 26.5 mm
- net Net-(C8-Pad2): track 16.3 -> 26.0 mm
- net Net-(C6-Pad2): track 18.8 -> 27.4 mm
- net Net-(C5-Pad1): track 20.1 -> 27.6 mm
- net RX: track 22.4 -> 29.8 mm
- net Net-(C7-Pad2): track 26.5 -> 20.6 mm
- net Net-(C6-Pad1): track 3.81 -> 7.40 mm
- net Net-(D2-Pad2): track 7.93 -> 5.08 mm
- net HF_2: track 19.0 -> 21.6 mm
- net Net-(C5-Pad2): track 5.61 -> 6.88 mm
- net Net-(D1-Pad2): track 3.81 -> 5.08 mm
- net Net-(C4-Pad1): track 9.94 -> 8.89 mm
- net HF_1: track 21.2 -> 20.3 mm
Other:
- board size 60 x 50 mm -> 75 x 50 mm
- net class Default: clearance 0.3 -> 0.2
- rule trace_clearance: 0.3 -> 0.2
- board text removed: "F4HYU"

Commit message: Commit
Commit
Parts:
- removed G***: LOGO, logos:F4HYU-6x3-Logo
- H1, H2, H3, H4: footprint alex-library:M3-Real-Hole -> alex-library:M3-Hole
- moved D2 12.0 mm to (118.1, 76.2)
- moved J3 11.4 mm to (162.6, 82.5)
- moved R7 10.9 mm to (114.3, 73.7)
- moved C5 10.2 mm to (146.1, 91.4)
- moved C7 10.2 mm to (146.1, 78.7)
- moved C8 10.2 mm to (146.1, 82.5)
- moved R1 10.2 mm to (156.2, 55.9)
- moved H2 10.0 mm to (165.0, 95.0)
- moved H4 10.0 mm to (165.0, 55.0)
- moved R2 9.92 mm to (110.5, 88.9)
- moved Q1 8.89 mm to (139.7, 74.9)
- moved R12 8.89 mm to (141.0, 87.6)
- moved R4 8.89 mm to (141.0, 95.2)
- moved R9 8.89 mm to (141.0, 91.4)
- moved R10 8.89 mm to (125.7, 83.8)
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Routing:
- net TX: track 72.2 -> 60.1 mm
- net Net-(C8-Pad2): track 26.0 -> 22.2 mm
- net RX: track 29.8 -> 26.8 mm
- net Net-(C1-Pad1): track 26.5 -> 24.1 mm
- net Net-(C5-Pad1): track 27.6 -> 25.3 mm
- net HF_1: track 20.3 -> 18.6 mm
- net Net-(C6-Pad2): track 27.4 -> 25.8 mm
- net Net-(D2-Pad2): track 5.08 -> 3.81 mm
- net HF_2: track 21.6 -> 20.3 mm
- net Net-(C6-Pad1): track 7.40 -> 6.13 mm
- net Net-(D1-Pad2): track 5.08 -> 3.81 mm
- net Net-(C5-Pad2): track 6.88 -> 5.61 mm
- net Net-(C4-Pad1): track 8.89 -> 8.15 mm
Other:
- board size 75 x 50 mm -> 65 x 50 mm
