File: Kicad/Module_2-Amplificateur_bi_directionel_-BITX40-Mod_21_22_23/Module_2-Amplificateur_bi_directionel_-BITX40-Mod_21_22_23.sch (KiCad schematic (older format))
At the start: 31 parts, among them J1 Conn_01x03, J2 Conn_01x02, J3 Conn_01x02, Q1 2N2222a, Q2 2N2222a

Commit message: Commit
Commit
Parts:
- H1, H2, H3, H4: footprint alex-library:M3-Real-Hole -> alex-library:M3-Hole
Changed lines of the file:
@@
 F 0 "H1" H 9050 1100 60  0001 C CNN
 F 1 "M3-Hole" H 9100 1400 60  0001 C CNN
-F 2 "alex-library:M3-Real-Hole" H 9100 1300 60  0001 C CNN
+F 2 "alex-library:M3-Hole" H 9100 1300 60  0001 C CNN
 F 3 "" H 9050 1250 60  0001 C CNN
 	1    9050 1250
@@
 F 0 "H2" H 9350 1100 60  0001 C CNN
 F 1 "M3-Hole" H 9400 1400 60  0001 C CNN
-F 2 "alex-library:M3-Real-Hole" H 9400 1300 60  0001 C CNN
+F 2 "alex-library:M3-Hole" H 9400 1300 60  0001 C CNN
 F 3 "" H 9350 1250 60  0001 C CNN
 	1    9350 1250
@@
 F 0 "H3" H 9650 1100 60  0001 C CNN
 F 1 "M3-Hole" H 9700 1400 60  0001 C CNN
-F 2 "alex-library:M3-Real-Hole" H 9700 1300 60  0001 C CNN
+F 2 "alex-library:M3-Hole" H 9700 1300 60  0001 C CNN
 F 3 "" H 9650 1250 60  0001 C CNN
 	1    9650 1250
@@
 F 0 "H4" H 9950 1100 60  0001 C CNN
 F 1 "M3-Hole" H 10000 1400 60  0001 C CNN
-F 2 "alex-library:M3-Real-Hole" H 10000 1300 60  0001 C CNN
+F 2 "alex-library:M3-Hole" H 10000 1300 60  0001 C CNN
 F 3 "" H 9950 1250 60  0001 C CNN
 	1    9950 1250
